Commit message: NameSpace change

File: assembled/urdf/assembled.urdf (robot description, URDF)
Before this commit: robot Aseembled.SLDASM, 7 links, 6 joints
Links:
- link DockingPlate1: geometry collision mesh filename=package://assembled/meshes/DockingPlate1.STL; visual mesh filename=package://assembled/meshes/DockingPlate1.STL
- link DockingPlate2: geometry collision mesh filename=package://assembled/meshes/DockingPlate2.STL; visual mesh filename=package://assembled/meshes/DockingPlate2.STL
- link Servo1: geometry collision mesh filename=package://assembled/meshes/Servo1.STL; visual mesh filename=package://assembled/meshes/Servo1.STL
- link Servo2: geometry collision mesh filename=package://assembled/meshes/Servo2.STL; visual mesh filename=package://assembled/meshes/Servo2.STL
- link Wheel1: geometry collision mesh filename=package://assembled/meshes/Wheel1.STL; visual mesh filename=package://assembled/meshes/Wheel1.STL
- link Wheel2: geometry collision mesh filename=package://assembled/meshes/Wheel2.STL; visual mesh filename=package://assembled/meshes/Wheel2.STL
- link base_link: geometry collision mesh filename=package://assembled/meshes/base_link.STL; visual mesh filename=package://assembled/meshes/base_link.STL
