Commit message: Revolute errors

File: iota/urdf/iota.urdf (robot description, URDF)
Before this commit: robot iota, 28 links, 27 joints
Links:
- link r_panel: mass 0.00563834139292078 -> 0
- link ub_r_wheel: mass 0.000576666035103962 -> 0.00057667
- link uf_l_motor: mass 0.000645828982770904 -> 0.00064583
Joints:
- joint back_dock: limit (none) -> lower=0 upper=0 effort=0 velocity=0; origin xyz=-0.00534999999999996 0 -0.019059332034942 rpy=3.14159265358979 0 -0.626368079302037 -> xyz=-0.00535 0 -0.019059 rpy=3.1416 0 -0.62637; type continuous -> revolute
- joint db_l_wheel: limit (none) -> lower=0 upper=0 effort=0 velocity=0; type continuous -> revolute
- joint db_r_wheel: limit (none) -> lower=0 upper=0 effort=0 velocity=0; origin xyz=0 0 0.021 rpy=3.14159265358979 0 0.106028806705873 -> xyz=0 0 0.021 rpy=3.1416 0 0.10603; type continuous -> revolute
- joint df_l_wheel: limit (none) -> lower=0 upper=0 effort=0 velocity=0; origin xyz=0 0 0.021 rpy=0 0 0.88390039009553 -> xyz=0 0 0.021 rpy=0 0 0.8839; type continuous -> revolute
- joint df_r_wheel: limit (none) -> lower=0 upper=0 effort=0 velocity=0; origin xyz=0 0 0.021 rpy=3.14159265358979 0 1.46819705601191 -> xyz=0 0 0.021 rpy=3.1416 0 1.4682; type continuous -> revolute
- joint front_dock: limit (none) -> lower=0 upper=0 effort=0 velocity=0; origin xyz=-0.00535000000000001 0 -0.0190593320349418 rpy=3.14159265358979 0 0.173000373416657 -> xyz=-0.00535 0 -0.019059 rpy=3.1416 0 0.173; type continuous -> revolute
- joint front_servo: origin xyz=0.0034656966666195 -0.00820924646147805 0.0226525215937532 rpy=-1.57079632679489 1.51354276544107 1.57056578752365 -> xyz=0.0034657 -0.0082092 0.022653 rpy=-1.5708 1.5135 1.5706
- joint l_panel: origin xyz=-0.015594256799817 -0.0766777315109957 0.0338985670725845 rpy=1.5707963267949 0 0 -> xyz=-0.015594 -0.076678 0.033899 rpy=1.5708 0 0
- joint ub_l_motor: origin xyz=-0.0278596823124971 0.00550000000000001 -0.000160189778555461 rpy=0 0 0.0567673670058895 -> xyz=-0.02786 0.0055 -0.00016019 rpy=0 0 0.056767
- joint ub_l_wheel: limit (none) -> lower=0 upper=0 effort=0 velocity=0; origin xyz=0 0 0.021 rpy=0 0 -0.0567673670058895 -> xyz=0 0 0.021 rpy=0 0 -0.056767; type continuous -> revolute
- joint ub_r_wheel: limit (none) -> lower=0 upper=0 effort=0 velocity=0; origin xyz=0 0 0.021 rpy=-3.14159265358979 0 2.33553651872795 -> xyz=0 0 0.021 rpy=-3.1416 0 2.3355; type continuous -> revolute
- joint uf_l_wheel: limit (none) -> lower=0 upper=0 effort=0 velocity=0; origin xyz=0 0 0.021 rpy=0 0 -0.420760994096352 -> xyz=0 0 0.021 rpy=0 0 -0.42076; type continuous -> revolute
- joint uf_r_Wheel: limit (none) -> lower=0 upper=0 effort=0 velocity=0; origin xyz=0 0 0.021 rpy=3.14159265358979 0 -2.58049522466332 -> xyz=0 0 0.021 rpy=3.1416 0 -2.5805; type continuous -> revolute

Commit message: Colorized

File: iota/urdf/iota.urdf (robot description, URDF)
Before this commit: robot iota, 28 links, 27 joints
Links:
- link back_dock: mass 0.000967710002344181 -> 0.00096771
- link back_panel: mass 0.00231351779814661 -> 0.0023135
- link back_servo: mass 0.00677100575579448 -> 0.006771
- link base_link: mass 0.00774047849628879 -> 0.0077405
- link db_l_motor: mass 0.000645828982770904 -> 0.00064583
- link db_l_wheel: mass 0.000576666035103963 -> 0.00057667
- link db_r_motor: mass 0.000645828982770904 -> 0.00064583
- link db_r_wheel: mass 0.000576666035103962 -> 0.00057667
- link df_l_motor: mass 0.000645828982770904 -> 0.00064583
- link df_l_wheel: mass 0.000576666035103963 -> 0.00057667
- link df_r_motor: mass 0.000645828982770904 -> 0.00064583
- link df_r_wheel: mass 0.000576666035103962 -> 0.00057667
- link front_dock: mass 0.00096771000234418 -> 0.00096771
- link front_panel: mass 0.00230993788046124 -> 0.0023099
- link front_servo: mass 0.00677100577989105 -> 0.006771
- link l_panel: mass 0.00563834139292079 -> 0.0056383
- link lower_bracket: mass 0.000238824 -> 0.00023882
- link top_panel: mass 0.00796322972446395 -> 0.0079632
- link ub_l_motor: mass 0.000645828982770904 -> 0.00064583
- link ub_l_wheel: mass 0.000576666035103963 -> 0.00057667
- link ub_r_motor: mass 0.000645828982770904 -> 0.00064583
- link ub_r_wheel: mass 0.000576666035103962 -> 0.00057667
- link uf_l_motor: mass 0.000645828982770904 -> 0.00064583
- link uf_l_wheel: mass 0.000576666035103963 -> 0.00057667
- link uf_r_motor: mass 0.000645828982770904 -> 0.00064583
- link uf_r_wheel: mass 0.000576666035103962 -> 0.00057667
- link upper_bracket: mass 0.000238824 -> 0.00023882
