Commit message: Masses and meshes updated

File: iota/absolute/iota.urdf (robot description, URDF)
Before this commit: robot iota, 28 links, 27 joints
Links:
- link back_dock: geometry collision mesh filename=meshes/back_dock.STL; visual mesh filename=meshes/back_dock.STL
- link back_panel: geometry collision mesh filename=meshes/back_panel.STL; visual mesh filename=meshes/back_panel.STL
- link back_servo: geometry collision mesh filename=meshes/back_servo.STL; visual mesh filename=meshes/back_servo.STL
- link base_link: geometry collision mesh filename=meshes/base_link.STL; visual mesh filename=meshes/base_link.STL
- link db_l_motor: geometry collision mesh filename=meshes/db_l_motor.STL; visual mesh filename=meshes/db_l_motor.STL
- link db_l_wheel: geometry collision mesh filename=meshes/db_l_wheel.STL; visual mesh filename=meshes/db_l_wheel.STL
- link db_r_motor: geometry collision mesh filename=meshes/db_r_motor.STL; visual mesh filename=meshes/db_r_motor.STL
- link db_r_wheel: geometry collision mesh filename=meshes/db_r_wheel.STL; visual mesh filename=meshes/db_r_wheel.STL
- link df_l_motor: geometry collision mesh filename=meshes/df_l_motor.STL; visual mesh filename=meshes/df_l_motor.STL
- link df_l_wheel: geometry collision mesh filename=meshes/df_l_wheel.STL; visual mesh filename=meshes/df_l_wheel.STL
- link df_r_motor: geometry collision mesh filename=meshes/df_r_motor.STL; visual mesh filename=meshes/df_r_motor.STL
- link df_r_wheel: geometry collision mesh filename=meshes/df_r_wheel.STL; visual mesh filename=meshes/df_r_wheel.STL
- link front_dock: geometry collision mesh filename=meshes/front_dock.STL; visual mesh filename=meshes/front_dock.STL
- link front_panel: geometry collision mesh filename=meshes/front_panel.STL; visual mesh filename=meshes/front_panel.STL
- link front_servo: geometry collision mesh filename=meshes/front_servo.STL; visual mesh filename=meshes/front_servo.STL
- link l_panel: geometry collision mesh filename=meshes/l_panel.STL; visual mesh filename=meshes/l_panel.STL
- link lower_bracket: geometry collision mesh filename=meshes/lower_bracket.STL; visual mesh filename=meshes/lower_bracket.STL
- link r_panel: geometry collision mesh filename=meshes/r_panel.STL; visual mesh filename=meshes/r_panel.STL
- link top_panel: geometry collision mesh filename=meshes/top_panel.STL; visual mesh filename=meshes/top_panel.STL
- link ub_l_motor: geometry collision mesh filename=meshes/ub_l_motor.STL; visual mesh filename=meshes/ub_l_motor.STL
- link ub_l_wheel: geometry collision mesh filename=meshes/ub_l_wheel.STL; visual mesh filename=meshes/ub_l_wheel.STL
- link ub_r_motor: geometry collision mesh filename=meshes/ub_r_motor.STL; visual mesh filename=meshes/ub_r_motor.STL
- link ub_r_wheel: geometry collision mesh filename=meshes/ub_r_wheel.STL; visual mesh filename=meshes/ub_r_wheel.STL
- link uf_l_motor: geometry collision mesh filename=meshes/uf_l_motor.STL; visual mesh filename=meshes/uf_l_motor.STL
- link uf_l_wheel: geometry collision mesh filename=meshes/uf_l_wheel.STL; visual mesh filename=meshes/uf_l_wheel.STL
- link uf_r_motor: geometry collision mesh filename=meshes/uf_r_motor.STL; visual mesh filename=meshes/uf_r_motor.STL
- link uf_r_wheel: geometry collision mesh filename=meshes/uf_r_wheel.STL; visual mesh filename=meshes/uf_r_wheel.STL
- link upper_bracket: geometry collision mesh filename=meshes/upper_bracket.STL; visual mesh filename=meshes/upper_bracket.STL

Commit message: done simulation

File: iota/absolute/iota.urdf (robot description, URDF)
Before this commit: robot iota, 28 links, 27 joints
Links:
- link back_dock: geometry collision mesh filename=package://iota/meshes/back_dock.STL; visual mesh filename=package://iota/meshes/back_dock.STL
- link back_panel: geometry collision mesh filename=package://iota/meshes/back_panel.STL; visual mesh filename=package://iota/meshes/back_panel.STL
- link back_servo: geometry collision mesh filename=package://iota/meshes/back_servo.STL; visual mesh filename=package://iota/meshes/back_servo.STL
- link base_link: geometry collision mesh filename=package://iota/meshes/base_link.STL; visual mesh filename=package://iota/meshes/base_link.STL
- link db_l_motor: geometry collision mesh filename=package://iota/meshes/db_l_motor.STL; visual mesh filename=package://iota/meshes/db_l_motor.STL
- link db_l_wheel: geometry collision mesh filename=package://iota/meshes/db_l_wheel.STL; visual mesh filename=package://iota/meshes/db_l_wheel.STL
- link db_r_motor: geometry collision mesh filename=package://iota/meshes/db_r_motor.STL; visual mesh filename=package://iota/meshes/db_r_motor.STL
- link db_r_wheel: geometry collision mesh filename=package://iota/meshes/db_r_wheel.STL; visual mesh filename=package://iota/meshes/db_r_wheel.STL
- link df_l_motor: geometry collision mesh filename=package://iota/meshes/df_l_motor.STL; visual mesh filename=package://iota/meshes/df_l_motor.STL
- link df_l_wheel: geometry collision mesh filename=package://iota/meshes/df_l_wheel.STL; visual mesh filename=package://iota/meshes/df_l_wheel.STL
- link df_r_motor: geometry collision mesh filename=package://iota/meshes/df_r_motor.STL; visual mesh filename=package://iota/meshes/df_r_motor.STL
- link df_r_wheel: geometry collision mesh filename=package://iota/meshes/df_r_wheel.STL; visual mesh filename=package://iota/meshes/df_r_wheel.STL
- link front_dock: geometry collision mesh filename=package://iota/meshes/front_dock.STL; visual mesh filename=package://iota/meshes/front_dock.STL
- link front_panel: geometry collision mesh filename=package://iota/meshes/front_panel.STL; visual mesh filename=package://iota/meshes/front_panel.STL
- link front_servo: geometry collision mesh filename=package://iota/meshes/front_servo.STL; visual mesh filename=package://iota/meshes/front_servo.STL
- link l_panel: geometry collision mesh filename=package://iota/meshes/l_panel.STL; visual mesh filename=package://iota/meshes/l_panel.STL
- link lower_bracket: geometry collision mesh filename=package://iota/meshes/lower_bracket.STL; visual mesh filename=package://iota/meshes/lower_bracket.STL
- link r_panel: geometry collision mesh filename=package://iota/meshes/r_panel.STL; visual mesh filename=package://iota/meshes/r_panel.STL
- link top_panel: geometry collision mesh filename=package://iota/meshes/top_panel.STL; visual mesh filename=package://iota/meshes/top_panel.STL
- link ub_l_motor: geometry collision mesh filename=package://iota/meshes/ub_l_motor.STL; visual mesh filename=package://iota/meshes/ub_l_motor.STL
- link ub_l_wheel: geometry collision mesh filename=package://iota/meshes/ub_l_wheel.STL; visual mesh filename=package://iota/meshes/ub_l_wheel.STL
- link ub_r_motor: geometry collision mesh filename=package://iota/meshes/ub_r_motor.STL; visual mesh filename=package://iota/meshes/ub_r_motor.STL
- link ub_r_wheel: geometry collision mesh filename=package://iota/meshes/ub_r_wheel.STL; visual mesh filename=package://iota/meshes/ub_r_wheel.STL
- link uf_l_motor: geometry collision mesh filename=package://iota/meshes/uf_l_motor.STL; visual mesh filename=package://iota/meshes/uf_l_motor.STL
- link uf_l_wheel: geometry collision mesh filename=package://iota/meshes/uf_l_wheel.STL; visual mesh filename=package://iota/meshes/uf_l_wheel.STL
- link uf_r_motor: geometry collision mesh filename=package://iota/meshes/uf_r_motor.STL; visual mesh filename=package://iota/meshes/uf_r_motor.STL
- link uf_r_wheel: geometry collision mesh filename=package://iota/meshes/uf_r_wheel.STL; visual mesh filename=package://iota/meshes/uf_r_wheel.STL
- link upper_bracket: geometry collision mesh filename=package://iota/meshes/upper_bracket.STL; visual mesh filename=package://iota/meshes/upper_bracket.STL
Joints:
- joint back_dock: limit (none) -> lower=0 upper=0 effort=0 velocity=0
- joint db_l_wheel: limit (none) -> lower=0 upper=0 effort=0 velocity=0
- joint db_r_wheel: limit (none) -> lower=0 upper=0 effort=0 velocity=0
- joint df_l_wheel: limit (none) -> lower=0 upper=0 effort=0 velocity=0
- joint df_r_wheel: limit (none) -> lower=0 upper=0 effort=0 velocity=0
- joint front_dock: limit (none) -> lower=0 upper=0 effort=0 velocity=0
- joint ub_l_wheel: limit (none) -> lower=0 upper=0 effort=0 velocity=0
- joint ub_r_wheel: limit (none) -> lower=0 upper=0 effort=0 velocity=0
- joint uf_l_wheel: limit (none) -> lower=0 upper=0 effort=0 velocity=0
- joint uf_r_Wheel: limit (none) -> lower=0 upper=0 effort=0 velocity=0

File: iota/urdf/iota.urdf (robot description, URDF)
Before this commit: robot iota, 28 links, 27 joints
Links:
- link r_panel: mass 0 -> 0.00563834139292078
- link ub_r_wheel: mass 0.00057667 -> 0.000576666035103962
- link uf_l_motor: mass 0.00064583 -> 0.000645828982770904
Joints:
- joint back_dock: origin xyz=-0.00535 0 -0.019059 rpy=3.1416 0 -0.62637 -> xyz=-0.00534999999999996 0 -0.019059332034942 rpy=3.14159265358979 0 -0.626368079302037; type revolute -> continuous
- joint db_l_wheel: type revolute -> continuous
- joint db_r_wheel: origin xyz=0 0 0.021 rpy=3.1416 0 0.10603 -> xyz=0 0 0.021 rpy=3.14159265358979 0 0.106028806705873; type revolute -> continuous
- joint df_l_wheel: origin xyz=0 0 0.021 rpy=0 0 0.8839 -> xyz=0 0 0.021 rpy=0 0 0.88390039009553; type revolute -> continuous
- joint df_r_wheel: origin xyz=0 0 0.021 rpy=3.1416 0 1.4682 -> xyz=0 0 0.021 rpy=3.14159265358979 0 1.46819705601191; type revolute -> continuous
- joint front_dock: origin xyz=-0.00535 0 -0.019059 rpy=3.1416 0 0.173 -> xyz=-0.00535000000000001 0 -0.0190593320349418 rpy=3.14159265358979 0 0.173000373416657; type revolute -> continuous
- joint front_servo: origin xyz=0.0034657 -0.0082092 0.022653 rpy=-1.5708 1.5135 1.5706 -> xyz=0.0034656966666195 -0.00820924646147805 0.0226525215937532 rpy=-1.57079632679489 1.51354276544107 1.57056578752365
- joint l_panel: origin xyz=-0.015594 -0.076678 0.033899 rpy=1.5708 0 0 -> xyz=-0.015594256799817 -0.0766777315109957 0.0338985670725845 rpy=1.5707963267949 0 0
- joint ub_l_motor: origin xyz=-0.02786 0.0055 -0.00016019 rpy=0 0 0.056767 -> xyz=-0.0278596823124971 0.00550000000000001 -0.000160189778555461 rpy=0 0 0.0567673670058895
- joint ub_l_wheel: origin xyz=0 0 0.021 rpy=0 0 -0.056767 -> xyz=0 0 0.021 rpy=0 0 -0.0567673670058895; type revolute -> continuous
- joint ub_r_wheel: origin xyz=0 0 0.021 rpy=-3.1416 0 2.3355 -> xyz=0 0 0.021 rpy=-3.14159265358979 0 2.33553651872795; type revolute -> continuous
- joint uf_l_wheel: origin xyz=0 0 0.021 rpy=0 0 -0.42076 -> xyz=0 0 0.021 rpy=0 0 -0.420760994096352; type revolute -> continuous
- joint uf_r_Wheel: origin xyz=0 0 0.021 rpy=3.1416 0 -2.5805 -> xyz=0 0 0.021 rpy=3.14159265358979 0 -2.58049522466332; type revolute -> continuous

Commit message: Colorized

File: iota/absolute/iota.urdf (robot description, URDF)
Before this commit: robot iota, 28 links, 27 joints
Links:
- link back_dock: mass 0.000967710002344181 -> 0.00096771; geometry collision mesh filename=meshes/back_dock.STL; visual mesh filename=meshes/back_dock.STL
- link back_panel: mass 0.00231351779814661 -> 0.0023135; geometry collision mesh filename=meshes/back_panel.STL; visual mesh filename=meshes/back_panel.STL
- link back_servo: mass 0.00677100575579448 -> 0.006771; geometry collision mesh filename=meshes/back_servo.STL; visual mesh filename=meshes/back_servo.STL
- link base_link: mass 0.00774047849628879 -> 0.0077405; geometry collision mesh filename=meshes/base_link.STL; visual mesh filename=meshes/base_link.STL
- link db_l_motor: mass 0.000645828982770904 -> 0.00064583; geometry collision mesh filename=meshes/db_l_motor.STL; visual mesh filename=meshes/db_l_motor.STL
- link db_l_wheel: mass 0.000576666035103963 -> 0.00057667; geometry collision mesh filename=meshes/db_l_wheel.STL; visual mesh filename=meshes/db_l_wheel.STL
- link db_r_motor: mass 0.000645828982770904 -> 0.00064583; geometry collision mesh filename=meshes/db_r_motor.STL; visual mesh filename=meshes/db_r_motor.STL
- link db_r_wheel: mass 0.000576666035103962 -> 0.00057667; geometry collision mesh filename=meshes/db_r_wheel.STL; visual mesh filename=meshes/db_r_wheel.STL
- link df_l_motor: mass 0.000645828982770904 -> 0.00064583; geometry collision mesh filename=meshes/df_l_motor.STL; visual mesh filename=meshes/df_l_motor.STL
- link df_l_wheel: mass 0.000576666035103963 -> 0.00057667; geometry collision mesh filename=meshes/df_l_wheel.STL; visual mesh filename=meshes/df_l_wheel.STL
- link df_r_motor: mass 0.000645828982770904 -> 0.00064583; geometry collision mesh filename=meshes/df_r_motor.STL; visual mesh filename=meshes/df_r_motor.STL
- link df_r_wheel: mass 0.000576666035103962 -> 0.00057667; geometry collision mesh filename=meshes/df_r_wheel.STL; visual mesh filename=meshes/df_r_wheel.STL
- link front_dock: mass 0.00096771000234418 -> 0.00096771; geometry collision mesh filename=meshes/front_dock.STL; visual mesh filename=meshes/front_dock.STL
- link front_panel: mass 0.00230993788046124 -> 0.0023099; geometry collision mesh filename=meshes/front_panel.STL; visual mesh filename=meshes/front_panel.STL
- link front_servo: mass 0.00677100577989105 -> 0.006771; geometry collision mesh filename=meshes/front_servo.STL; visual mesh filename=meshes/front_servo.STL
- link l_panel: mass 0.00563834139292079 -> 0.0056383; geometry collision mesh filename=meshes/l_panel.STL; visual mesh filename=meshes/l_panel.STL
- link lower_bracket: mass 0.000238824 -> 0.00023882; geometry collision mesh filename=meshes/lower_bracket.STL; visual mesh filename=meshes/lower_bracket.STL
- link r_panel: geometry collision mesh filename=meshes/r_panel.STL; visual mesh filename=meshes/r_panel.STL
- link top_panel: mass 0.00796322972446395 -> 0.0079632; geometry collision mesh filename=meshes/top_panel.STL; visual mesh filename=meshes/top_panel.STL
- link ub_l_motor: mass 0.000645828982770904 -> 0.00064583; geometry collision mesh filename=meshes/ub_l_motor.STL; visual mesh filename=meshes/ub_l_motor.STL
- link ub_l_wheel: mass 0.000576666035103963 -> 0.00057667; geometry collision mesh filename=meshes/ub_l_wheel.STL; visual mesh filename=meshes/ub_l_wheel.STL
- link ub_r_motor: mass 0.000645828982770904 -> 0.00064583; geometry collision mesh filename=meshes/ub_r_motor.STL; visual mesh filename=meshes/ub_r_motor.STL
- link ub_r_wheel: mass 0.000576666035103962 -> 0.00057667; geometry collision mesh filename=meshes/ub_r_wheel.STL; visual mesh filename=meshes/ub_r_wheel.STL
- link uf_l_motor: mass 0.000645828982770904 -> 0.00064583; geometry collision mesh filename=meshes/uf_l_motor.STL; visual mesh filename=meshes/uf_l_motor.STL
- link uf_l_wheel: mass 0.000576666035103963 -> 0.00057667; geometry collision mesh filename=meshes/uf_l_wheel.STL; visual mesh filename=meshes/uf_l_wheel.STL
- link uf_r_motor: mass 0.000645828982770904 -> 0.00064583; geometry collision mesh filename=meshes/uf_r_motor.STL; visual mesh filename=meshes/uf_r_motor.STL
- link uf_r_wheel: mass 0.000576666035103962 -> 0.00057667; geometry collision mesh filename=meshes/uf_r_wheel.STL; visual mesh filename=meshes/uf_r_wheel.STL
- link upper_bracket: mass 0.000238824 -> 0.00023882; geometry collision mesh filename=meshes/upper_bracket.STL; visual mesh filename=meshes/upper_bracket.STL
