Commit message: Docking mechanism

File: iota/absolute/iota.urdf (robot description, URDF)
Before this commit: robot iota, 28 links, 27 joints
Links:
- removed link back_dock
- removed link back_panel
- removed link back_servo
- removed link db_l_motor
- removed link db_l_wheel
- removed link db_r_motor
- removed link db_r_wheel
- removed link df_l_motor
- removed link df_l_wheel
- removed link df_r_motor
- removed link df_r_wheel
- removed link front_dock
- removed link front_panel
- removed link front_servo
- removed link l_panel
- removed link lower_bracket
- removed link r_panel
- removed link top_panel
- removed link ub_l_motor
- removed link ub_l_wheel
- removed link ub_r_motor
- removed link ub_r_wheel
- removed link uf_l_motor
- removed link uf_l_wheel
- removed link uf_r_motor
- removed link uf_r_wheel
- removed link upper_bracket
- added link b_dock, mass 0.000956519229010847; collision mesh filename=meshes/b_dock.STL; visual mesh filename=meshes/b_dock.STL
- added link b_plate, mass 0.00230993788046124; collision mesh filename=meshes/b_plate.STL; visual mesh filename=meshes/b_plate.STL
- added link b_servo, mass 0.00677100577989105; collision mesh filename=meshes/b_servo.STL; visual mesh filename=meshes/b_servo.STL
- added link dbl_motor, mass 0.000645828982770904; collision mesh filename=meshes/dbl_motor.STL; visual mesh filename=meshes/dbl_motor.STL
- added link dbl_wheel, mass 0.000681713039458372; collision mesh filename=meshes/dbl_wheel.STL; visual mesh filename=meshes/dbl_wheel.STL
- added link dbr_motor, mass 0.000645828982770904; collision mesh filename=meshes/dbr_motor.STL; visual mesh filename=meshes/dbr_motor.STL
- added link dbr_wheel, mass 0.000681713039458371; collision mesh filename=meshes/dbr_wheel.STL; visual mesh filename=meshes/dbr_wheel.STL
- added link dfl_motor, mass 0.000645828982770904; collision mesh filename=meshes/dfl_motor.STL; visual mesh filename=meshes/dfl_motor.STL
- added link dfl_wheel, mass 0.000681713039458372; collision mesh filename=meshes/dfl_wheel.STL; visual mesh filename=meshes/dfl_wheel.STL
- added link dfr_motor, mass 0.000645828982770904; collision mesh filename=meshes/dfr_motor.STL; visual mesh filename=meshes/dfr_motor.STL
- added link dfr_wheel, mass 0.000681713039458371; collision mesh filename=meshes/dfr_wheel.STL; visual mesh filename=meshes/dfr_wheel.STL
- added link f_dock, mass 0.000956519229010847; collision mesh filename=meshes/f_dock.STL; visual mesh filename=meshes/f_dock.STL
- added link f_plate, mass 0.00231351779814661; collision mesh filename=meshes/f_plate.STL; visual mesh filename=meshes/f_plate.STL
- added link f_servo, mass 0.00677100575579448; collision mesh filename=meshes/f_servo.STL; visual mesh filename=meshes/f_servo.STL
- added link l_plate, mass 0.00563834139292079; collision mesh filename=meshes/l_plate.STL; visual mesh filename=meshes/l_plate.STL
- added link lower_pin, mass 0.000238824; collision mesh filename=meshes/lower_pin.STL; visual mesh filename=meshes/lower_pin.STL
- added link r_plate, mass 0.00563834139292078; collision mesh filename=meshes/r_plate.STL; visual mesh filename=meshes/r_plate.STL
- added link tbl_motor, mass 0.000645828982770904; collision mesh filename=meshes/tbl_motor.STL; visual mesh filename=meshes/tbl_motor.STL
- added link tbl_wheel, mass 0.000681713039458371; collision mesh filename=meshes/tbl_wheel.STL; visual mesh filename=meshes/tbl_wheel.STL
- added link tbr_motor, mass 0.000645828982770904; collision mesh filename=meshes/tbr_motor.STL; visual mesh filename=meshes/tbr_motor.STL
- added link tbr_wheel, mass 0.000681713039458371; collision mesh filename=meshes/tbr_wheel.STL; visual mesh filename=meshes/tbr_wheel.STL
- added link tfl_motor, mass 0.000645828982770904; collision mesh filename=meshes/tfl_motor.STL; visual mesh filename=meshes/tfl_motor.STL
- added link tfl_wheel, mass 0.000681713039458372; collision mesh filename=meshes/tfl_wheel.STL; visual mesh filename=meshes/tfl_wheel.STL
- added link tfr_motor, mass 0.000645828982770904; collision mesh filename=meshes/tfr_motor.STL; visual mesh filename=meshes/tfr_motor.STL
- added link tfr_wheel, mass 0.000681713039458371; collision mesh filename=meshes/tfr_wheel.STL; visual mesh filename=meshes/tfr_wheel.STL
- added link top_plate, mass 0.00602026632101009; collision mesh filename=meshes/top_plate.STL; visual mesh filename=meshes/top_plate.STL
- added link upper_pin, mass 0.000238824; collision mesh filename=meshes/upper_pin.STL; visual mesh filename=meshes/upper_pin.STL
- link base_link: mass 0.0077405 -> 0.00602026598183142
Joints:
- removed joint back_dock
- removed joint back_panel
- removed joint back_servo
- removed joint db_l_motor
- removed joint db_l_wheel
- removed joint db_r_motor
- removed joint db_r_wheel
- removed joint df_l_motor
- removed joint df_l_wheel
- removed joint df_r_motor
- removed joint df_r_wheel
- removed joint front_dock
- removed joint front_panel
- removed joint front_servo
- removed joint l_panel
- removed joint lower_bracket
- removed joint r_panel
- removed joint top_panel
- removed joint ub_l_motor
- removed joint ub_l_wheel
- removed joint ub_r_motor
- removed joint ub_r_wheel
- removed joint uf_l_motor
- removed joint uf_l_wheel
- removed joint uf_r_Wheel
- removed joint uf_r_motor
- removed joint upper_bracket
- added joint b_dock: type continuous, parent b_servo, child b_dock, origin xyz=-0.00535000000000001 0 -0.0215593320349418 rpy=3.14159265358979 0 -2.35638402492922, axis 0 0 1
- added joint b_plate: type fixed, parent l_plate, child b_plate, origin xyz=0.06388 0.020927 -0.02875 rpy=-1.3638 1.5708 -1.5667, axis 0 0 0
- added joint b_servo: type fixed, parent upper_pin, child b_servo, origin xyz=0.0034656966666195 -0.00820924646147805 0.0226525215937532 rpy=-1.57079632679489 1.51354276544107 1.57056578752365, axis 0 0 0
- added joint dbl_motor: type fixed, parent base_link, child dbl_motor, origin xyz=0.0337512124928369 -0.0488651262442055 0.0368985670725845 rpy=1.5707963267949 -0.344784457208072 0, axis 0 0 0
- added joint dbl_wheel: type continuous, parent dbl_motor, child dbl_wheel, origin xyz=0 0 0.021 rpy=0 0 -0.528472588992204, axis 0 0 1
- added joint dbr_motor: type fixed, parent base_link, child dbr_motor, origin xyz=0.0157046714219995 -0.0486777315109957 0.0313985670725845 rpy=1.5707963267949 0 0, axis 0 0 0
- added joint dbr_wheel: type continuous, parent dbr_motor, child dbr_wheel, origin xyz=0.0180465410708374 0.0055 -0.0258126052667903 rpy=0 0 -0.151232003284142, axis 0 0 1
- added joint dfl_motor: type fixed, parent base_link, child dfl_motor, origin xyz=-0.00164838652382185 -0.0491355291275451 0.0368985670725845 rpy=1.5707963267949 -0.0567673670058903 0, axis 0 0 0
- added joint dfl_wheel: type continuous, parent dfl_motor, child dfl_wheel, origin xyz=0 0 0.021 rpy=0 0 -0.0567673670058903, axis 0 0 1
- added joint dfr_motor: type fixed, parent base_link, child dfr_motor, origin xyz=-0.00164838652382185 -0.0491355291275451 0.0368985670725845 rpy=1.5707963267949 -0.890920085389358 3.14159265358979, axis 0 0 0
- added joint dfr_wheel: type continuous, parent dfr_motor, child dfr_wheel, origin xyz=0 0 0.021 rpy=3.14159265358979 0 2.42846104804575, axis 0 0 1
- added joint f_dock: type continuous, parent f_servo, child f_dock, origin xyz=-0.00534999999999996 0 -0.0215593320349417 rpy=3.14159265358979 0 3.03104582528322, axis 0 0 1
- added joint f_plate: type fixed, parent r_plate, child f_plate, origin xyz=0.00710981547880829 0.0247871496673297 0.02925 rpy=0.279335238189619 1.5707963267949 0, axis 0 0 0
- added joint f_servo: type fixed, parent lower_pin, child f_servo, origin xyz=-0.00327850155878186 0.00710820887028432 0.0211565538865111 rpy=0 1.5707963267949 0, axis 0 0 0
- added joint l_plate: type fixed, parent base_link, child l_plate, origin xyz=-0.015594256799817 -0.0766777315109957 0.0338985670725845 rpy=1.5707963267949 0 0, axis 0 0 0
- added joint lower_pin: type fixed, parent r_plate, child lower_pin, origin xyz=0.028589 0.013247 0.0031239 rpy=0.057254 0 -0.27933, axis 0 0 0
- added joint r_plate: type fixed, parent base_link, child r_plate, origin xyz=-0.0156361653843612 -0.0186777315109957 0.0338985670725845 rpy=1.5707963267949 0 0, axis 0 0 0
- added joint tbl_motor: type fixed, parent top_plate, child tbl_motor, origin xyz=0.0178826765348059 -0.00299999999999999 -0.000144283776645951 rpy=0 0 -0.997183454252289, axis 0 0 1
- added joint tbl_wheel: type continuous, parent tbl_motor, child tbl_wheel, origin xyz=0 0 0.021 rpy=0 0 1.10845521806602, axis 0 0 1
- added joint tbr_motor: type fixed, parent top_plate, child tbr_motor, origin xyz=0.0178826765348059 -0.00299999999999999 -0.000144283776645951 rpy=3.14159265358979 0 1.46819705601191, axis 0 0 0
- added joint tbr_wheel: type continuous, parent tbr_motor, child tbr_wheel, origin xyz=0 0 0.021 rpy=3.1416 0 1.4682, axis 0 0 1
- added joint tfl_motor: type fixed, parent top_plate, child tfl_motor, origin xyz=-0.0194941929617864 -0.003 -2.24534021392858E-05 rpy=0 0 0, axis 0 0 0
- added joint tfl_wheel: type continuous, parent tfl_motor, child tfl_wheel, origin xyz=0 0 0.021 rpy=0 0 0, axis 0 0 1
- added joint tfr_motor: type fixed, parent top_plate, child tfr_motor, origin xyz=-0.0194941929617864 -0.003 -2.24534021392858E-05 rpy=3.14159265358979 0 0.106028806705873, axis 0 0 1
- added joint tfr_wheel: type continuous, parent tfr_motor, child tfr_wheel, origin xyz=0 0 0.021 rpy=3.14159265358979 0 0.106028806705873, axis 0 0 1
- added joint top_plate: type fixed, parent l_plate, child top_plate, origin xyz=0.042248384032793 0.045 -0.028 rpy=0 0 0, axis 0 0 0
- added joint upper_pin: type fixed, parent l_plate, child upper_pin, origin xyz=0.045176 0.035576 -0.056 rpy=0 0 -0.2791, axis 0 0 0

File: iota/urdf/iota.urdf (robot description, URDF)
Before this commit: robot iota, 28 links, 27 joints
Links:
- removed link back_dock
- removed link back_panel
- removed link back_servo
- removed link db_l_motor
- removed link db_l_wheel
- removed link db_r_motor
- removed link db_r_wheel
- removed link df_l_motor
- removed link df_l_wheel
- removed link df_r_motor
- removed link df_r_wheel
- removed link front_dock
- removed link front_panel
- removed link front_servo
- removed link l_panel
- removed link lower_bracket
- removed link r_panel
- removed link top_panel
- removed link ub_l_motor
- removed link ub_l_wheel
- removed link ub_r_motor
- removed link ub_r_wheel
- removed link uf_l_motor
- removed link uf_l_wheel
- removed link uf_r_motor
- removed link uf_r_wheel
- removed link upper_bracket
- added link b_dock, mass 0.000956519229010847; collision mesh filename=package://iota/meshes/b_dock.STL; visual mesh filename=package://iota/meshes/b_dock.STL
- added link b_plate, mass 0.00230993788046124; collision mesh filename=package://iota/meshes/b_plate.STL; visual mesh filename=package://iota/meshes/b_plate.STL
- added link b_servo, mass 0.00677100577989105; collision mesh filename=package://iota/meshes/b_servo.STL; visual mesh filename=package://iota/meshes/b_servo.STL
- added link dbl_motor, mass 0.000645828982770904; collision mesh filename=package://iota/meshes/dbl_motor.STL; visual mesh filename=package://iota/meshes/dbl_motor.STL
- added link dbl_wheel, mass 0.000681713039458372; collision mesh filename=package://iota/meshes/dbl_wheel.STL; visual mesh filename=package://iota/meshes/dbl_wheel.STL
- added link dbr_motor, mass 0.000645828982770904; collision mesh filename=package://iota/meshes/dbr_motor.STL; visual mesh filename=package://iota/meshes/dbr_motor.STL
- added link dbr_wheel, mass 0.000681713039458371; collision mesh filename=package://iota/meshes/dbr_wheel.STL; visual mesh filename=package://iota/meshes/dbr_wheel.STL
- added link dfl_motor, mass 0.000645828982770904; collision mesh filename=package://iota/meshes/dfl_motor.STL; visual mesh filename=package://iota/meshes/dfl_motor.STL
- added link dfl_wheel, mass 0.000681713039458372; collision mesh filename=package://iota/meshes/dfl_wheel.STL; visual mesh filename=package://iota/meshes/dfl_wheel.STL
- added link dfr_motor, mass 0.000645828982770904; collision mesh filename=package://iota/meshes/dfr_motor.STL; visual mesh filename=package://iota/meshes/dfr_motor.STL
- added link dfr_wheel, mass 0.000681713039458371; collision mesh filename=package://iota/meshes/dfr_wheel.STL; visual mesh filename=package://iota/meshes/dfr_wheel.STL
- added link f_dock, mass 0.000956519229010847; collision mesh filename=package://iota/meshes/f_dock.STL; visual mesh filename=package://iota/meshes/f_dock.STL
- added link f_plate, mass 0.00231351779814661; collision mesh filename=package://iota/meshes/f_plate.STL; visual mesh filename=package://iota/meshes/f_plate.STL
- added link f_servo, mass 0.00677100575579448; collision mesh filename=package://iota/meshes/f_servo.STL; visual mesh filename=package://iota/meshes/f_servo.STL
- added link l_plate, mass 0.00563834139292079; collision mesh filename=package://iota/meshes/l_plate.STL; visual mesh filename=package://iota/meshes/l_plate.STL
- added link lower_pin, mass 0.000238824; collision mesh filename=package://iota/meshes/lower_pin.STL; visual mesh filename=package://iota/meshes/lower_pin.STL
- added link r_plate, mass 0.00563834139292078; collision mesh filename=package://iota/meshes/r_plate.STL; visual mesh filename=package://iota/meshes/r_plate.STL
- added link tbl_motor, mass 0.000645828982770904; collision mesh filename=package://iota/meshes/tbl_motor.STL; visual mesh filename=package://iota/meshes/tbl_motor.STL
- added link tbl_wheel, mass 0.000681713039458371; collision mesh filename=package://iota/meshes/tbl_wheel.STL; visual mesh filename=package://iota/meshes/tbl_wheel.STL
- added link tbr_motor, mass 0.000645828982770904; collision mesh filename=package://iota/meshes/tbr_motor.STL; visual mesh filename=package://iota/meshes/tbr_motor.STL
- added link tbr_wheel, mass 0.000681713039458371; collision mesh filename=package://iota/meshes/tbr_wheel.STL; visual mesh filename=package://iota/meshes/tbr_wheel.STL
- added link tfl_motor, mass 0.000645828982770904; collision mesh filename=package://iota/meshes/tfl_motor.STL; visual mesh filename=package://iota/meshes/tfl_motor.STL
- added link tfl_wheel, mass 0.000681713039458372; collision mesh filename=package://iota/meshes/tfl_wheel.STL; visual mesh filename=package://iota/meshes/tfl_wheel.STL
- added link tfr_motor, mass 0.000645828982770904; collision mesh filename=package://iota/meshes/tfr_motor.STL; visual mesh filename=package://iota/meshes/tfr_motor.STL
- added link tfr_wheel, mass 0.000681713039458371; collision mesh filename=package://iota/meshes/tfr_wheel.STL; visual mesh filename=package://iota/meshes/tfr_wheel.STL
- added link top_plate, mass 0.00602026632101009; collision mesh filename=package://iota/meshes/top_plate.STL; visual mesh filename=package://iota/meshes/top_plate.STL
- added link upper_pin, mass 0.000238824; collision mesh filename=package://iota/meshes/upper_pin.STL; visual mesh filename=package://iota/meshes/upper_pin.STL
- link base_link: mass 0.0077405 -> 0.00602026598183142
Joints:
- removed joint back_dock
- removed joint back_panel
- removed joint back_servo
- removed joint db_l_motor
- removed joint db_l_wheel
- removed joint db_r_motor
- removed joint db_r_wheel
- removed joint df_l_motor
- removed joint df_l_wheel
- removed joint df_r_motor
- removed joint df_r_wheel
- removed joint front_dock
- removed joint front_panel
- removed joint front_servo
- removed joint l_panel
- removed joint lower_bracket
- removed joint r_panel
- removed joint top_panel
- removed joint ub_l_motor
- removed joint ub_l_wheel
- removed joint ub_r_motor
- removed joint ub_r_wheel
- removed joint uf_l_motor
- removed joint uf_l_wheel
- removed joint uf_r_Wheel
- removed joint uf_r_motor
- removed joint upper_bracket
- added joint b_dock: type continuous, parent b_servo, child b_dock, origin xyz=-0.00535000000000001 0 -0.0215593320349418 rpy=3.14159265358979 0 -2.35638402492922, axis 0 0 1
- added joint b_plate: type fixed, parent l_plate, child b_plate, origin xyz=0.06388 0.020927 -0.02875 rpy=-1.3638 1.5708 -1.5667, axis 0 0 0
- added joint b_servo: type fixed, parent upper_pin, child b_servo, origin xyz=0.0034656966666195 -0.00820924646147805 0.0226525215937532 rpy=-1.57079632679489 1.51354276544107 1.57056578752365, axis 0 0 0
- added joint dbl_motor: type fixed, parent base_link, child dbl_motor, origin xyz=0.0337512124928369 -0.0488651262442055 0.0368985670725845 rpy=1.5707963267949 -0.344784457208072 0, axis 0 0 0
- added joint dbl_wheel: type continuous, parent dbl_motor, child dbl_wheel, origin xyz=0 0 0.021 rpy=0 0 -0.528472588992204, axis 0 0 1
- added joint dbr_motor: type fixed, parent base_link, child dbr_motor, origin xyz=0.0157046714219995 -0.0486777315109957 0.0313985670725845 rpy=1.5707963267949 0 0, axis 0 0 0
- added joint dbr_wheel: type continuous, parent dbr_motor, child dbr_wheel, origin xyz=0.0180465410708374 0.0055 -0.0258126052667903 rpy=0 0 -0.151232003284142, axis 0 0 1
- added joint dfl_motor: type fixed, parent base_link, child dfl_motor, origin xyz=-0.00164838652382185 -0.0491355291275451 0.0368985670725845 rpy=1.5707963267949 -0.0567673670058903 0, axis 0 0 0
- added joint dfl_wheel: type continuous, parent dfl_motor, child dfl_wheel, origin xyz=0 0 0.021 rpy=0 0 -0.0567673670058903, axis 0 0 1
- added joint dfr_motor: type fixed, parent base_link, child dfr_motor, origin xyz=-0.00164838652382185 -0.0491355291275451 0.0368985670725845 rpy=1.5707963267949 -0.890920085389358 3.14159265358979, axis 0 0 0
- added joint dfr_wheel: type continuous, parent dfr_motor, child dfr_wheel, origin xyz=0 0 0.021 rpy=3.14159265358979 0 2.42846104804575, axis 0 0 1
- added joint f_dock: type continuous, parent f_servo, child f_dock, origin xyz=-0.00534999999999996 0 -0.0215593320349417 rpy=3.14159265358979 0 3.03104582528322, axis 0 0 1
- added joint f_plate: type fixed, parent r_plate, child f_plate, origin xyz=0.00710981547880829 0.0247871496673297 0.02925 rpy=0.279335238189619 1.5707963267949 0, axis 0 0 0
- added joint f_servo: type fixed, parent lower_pin, child f_servo, origin xyz=-0.00327850155878186 0.00710820887028432 0.0211565538865111 rpy=0 1.5707963267949 0, axis 0 0 0
- added joint l_plate: type fixed, parent base_link, child l_plate, origin xyz=-0.015594256799817 -0.0766777315109957 0.0338985670725845 rpy=1.5707963267949 0 0, axis 0 0 0
- added joint lower_pin: type fixed, parent r_plate, child lower_pin, origin xyz=0.028589 0.013247 0.0031239 rpy=0.057254 0 -0.27933, axis 0 0 0
- added joint r_plate: type fixed, parent base_link, child r_plate, origin xyz=-0.0156361653843612 -0.0186777315109957 0.0338985670725845 rpy=1.5707963267949 0 0, axis 0 0 0
- added joint tbl_motor: type fixed, parent top_plate, child tbl_motor, origin xyz=0.0178826765348059 -0.00299999999999999 -0.000144283776645951 rpy=0 0 -0.997183454252289, axis 0 0 1
- added joint tbl_wheel: type continuous, parent tbl_motor, child tbl_wheel, origin xyz=0 0 0.021 rpy=0 0 1.10845521806602, axis 0 0 1
- added joint tbr_motor: type fixed, parent top_plate, child tbr_motor, origin xyz=0.0178826765348059 -0.00299999999999999 -0.000144283776645951 rpy=3.14159265358979 0 1.46819705601191, axis 0 0 0
- added joint tbr_wheel: type continuous, parent tbr_motor, child tbr_wheel, origin xyz=0 0 0.021 rpy=3.1416 0 1.4682, axis 0 0 1
- added joint tfl_motor: type fixed, parent top_plate, child tfl_motor, origin xyz=-0.0194941929617864 -0.003 -2.24534021392858E-05 rpy=0 0 0, axis 0 0 0
- added joint tfl_wheel: type continuous, parent tfl_motor, child tfl_wheel, origin xyz=0 0 0.021 rpy=0 0 0, axis 0 0 1
- added joint tfr_motor: type fixed, parent top_plate, child tfr_motor, origin xyz=-0.0194941929617864 -0.003 -2.24534021392858E-05 rpy=3.14159265358979 0 0.106028806705873, axis 0 0 1
- added joint tfr_wheel: type continuous, parent tfr_motor, child tfr_wheel, origin xyz=0 0 0.021 rpy=3.14159265358979 0 0.106028806705873, axis 0 0 1
- added joint top_plate: type fixed, parent l_plate, child top_plate, origin xyz=0.042248384032793 0.045 -0.028 rpy=0 0 0, axis 0 0 0
- added joint upper_pin: type fixed, parent l_plate, child upper_pin, origin xyz=0.045176 0.035576 -0.056 rpy=0 0 -0.2791, axis 0 0 0
